File: kicad/AudioFilter.kicad_sch (KiCad schematic)
At the start: 62 parts, among them J1 Conn_01x02_Pin, J10 Conn_01x02_Pin, J2 Conn_01x02_Pin, J3 Conn_01x02_Pin, J4 Conn_01x04_Pin, J5 Conn_01x02_Pin, J6 Conn_01x03_Pin, J7 Conn_01x04_Pin, J8 Conn_01x04_Pin, J9 Conn_01x07_Pin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

Commit message: Some tidying up
Parts:
- RV2: value R_Potentiometer_Dual -> C100K_Dual
- renumbered R21 to R20, R24 to R21, SW2 to SW2a1, SW3 to SW2b1, SW4 to SW2c1
Connections:
- net GND: now also J2.1 (Pin_1); no longer J2.2 (Pin_2)
- net P1.2: now also J2.2 (Pin_2); no longer J2.1 (Pin_1)
Other:
- moved on the sheet: J2
Changed lines of the file:
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@@
 	(wire
 		(pts
+			(xy 104.14 91.44) (xy 100.33 91.44)
+		)
+		(stroke
+			(width 0)
+			(type default)
+		)
+	)
+	(wire
+		(pts
 			(xy 85.09 143.51) (xy 85.09 144.78)
 		)
@@
 	(wire
 		(pts
-			(xy 104.14 88.9) (xy 104.14 85.09)
+			(xy 104.14 85.09) (xy 104.14 88.9)
 		)
 		(stroke
@@
 	(wire
 		(pts
+			(xy 100.33 88.9) (xy 104.14 88.9)
+		)
+		(stroke
+			(width 0)
+			(type default)
+		)
+	)
+	(wire
+		(pts
 			(xy 219.71 36.83) (xy 229.87 36.83)
 		)
@@
 	(wire
 		(pts
+			(xy 104.14 95.25) (xy 104.14 91.44)
+		)
+		(stroke
+			(width 0)
+			(type default)
+		)
+	)
+	(wire
+		(pts
 			(xy 104.14 69.85) (xy 104.14 67.31)
 		)
@@
 	(symbol
 		(lib_id "power:GND")
-		(at 104.14 91.44 0)
+		(at 104.14 95.25 0)
 		(unit 1)
 		(exclude_from_sim no)
@@
 		(fields_autoplaced yes)
 		(property "Reference" "#PWR03"
-			(at 104.14 97.79 0)
+			(at 104.14 101.6 0)
 			(effects
 				(font
@@
 		)
 		(property "Value" "GND"
-			(at 104.14 96.52 0)
+			(at 104.14 100.33 0)
 			(effects
 				(font
@@
 		)
 		(property "Footprint" ""
-			(at 104.14 91.44 0)
+			(at 104.14 95.25 0)
 			(effects
 				(font
@@
 		)
 		(property "Datasheet" ""
-			(at 104.14 91.44 0)
+			(at 104.14 95.25 0)
 			(effects
 				(font
@@
 		)
 		(property "Description" "Power symbol creates a global label with name \"GND\" , ground"
-			(at 104.14 91.44 0)
+			(at 104.14 95.25 0)
 			(effects
 				(font
@@
 			)
 		)
-		(property "Value" "R_Potentiometer_Dual"
-			(at 86.36 187.96 0)
+		(property "Value" "C100K_Dual"
+			(at 103.632 179.07 0)
 			(effects
 				(font
 					(size 1.27 1.27)
 				)
-				(hide yes)
 			)
 		)
@@
 	(symbol
 		(lib_id "Connector:Conn_01x02_Pin")
-		(at 99.06 88.9 0)
+		(at 95.25 91.44 0)
+		(mirror x)
 		(unit 1)
 		(exclude_from_sim no)
@@
 		(dnp no)
 		(property "Reference" "J2"
-			(at 97.028 90.424 0)
+			(at 93.218 89.916 0)
 			(effects
 				(font
@@
 		)
 		(property "Value" "Conn_01x02_Pin"
-			(at 99.695 86.36 0)
+			(at 95.885 93.98 0)
 			(effects
 				(font
@@
 		)
 		(property "Footprint" "Connector_Molex:Molex_KK-254_AE-6410-02A_1x02_P2.54mm_Vertical"
-			(at 99.06 88.9 0)
+			(at 95.25 91.44 0)
 			(effects
 				(font
@@
 		)
 		(property "Datasheet" "~"
-			(at 99.06 88.9 0)
+			(at 95.25 91.44 0)
 			(effects
 				(font
@@
 		)
 		(property "Description" "Generic connector, single row, 01x02, script generated"
-			(at 99.06 88.9 0)
+			(at 95.25 91.44 0)
 			(effects
 				(font
@@
 		(on_board no)
 		(dnp no)
-		(property "Reference" "SW2"
+		(property "Reference" "SW2a1"
 			(at 27.94 32.766 0)
 			(effects
@@
 			(project ""
 				(path "/14ff44ab-002e-411d-9096-19b5f402ce82"
-					(reference "SW2")
+					(reference "SW2a1")
 					(unit 1)
 				)
@@
 		(on_board yes)
 		(dnp no)
-		(property "Reference" "R24"
+		(property "Reference" "R21"
 			(at 228.6 137.414 90)
 			(effects
@@
 			(project "AudioFilter"
 				(path "/14ff44ab-002e-411d-9096-19b5f402ce82"
-					(reference "R24")
+					(reference "R21")
 					(unit 1)
 				)
@@
 		(on_board no)
 		(dnp no)
-		(property "Reference" "SW4"
+		(property "Reference" "SW2c1"
 			(at 27.94 105.156 0)
 			(effects
@@
 			(project ""
 				(path "/14ff44ab-002e-411d-9096-19b5f402ce82"
-					(reference "SW4")
+					(reference "SW2c1")
 					(unit 1)
 				)
@@
 		(on_board yes)
 		(dnp no)
-		(property "Reference" "R21"
+		(property "Reference" "R20"
 			(at 215.646 151.892 0)
 			(effects
@@
 			(project ""
 				(path "/14ff44ab-002e-411d-9096-19b5f402ce82"
-					(reference "R21")
+					(reference "R20")
 					(unit 1)
 				)
@@
 		(on_board no)
 		(dnp no)
-		(property "Reference" "SW3"
+		(property "Reference" "SW2b1"
 			(at 27.94 67.056 0)
 			(effects
@@
 			(project ""
 				(path "/14ff44ab-002e-411d-9096-19b5f402ce82"
-					(reference "SW3")
+					(reference "SW2b1")
 					(unit 1)
 				)

Commit message: Component size adjustments
Parts:
- C1: value 1uF -> 1uF 16V A
- C10, C9: value 10uF -> 10uF 16V
- C11: value 47pF -> 47pF PP; footprint Capacitor_THT:C_Disc_D5.0mm_W2.5mm_P5.00mm -> Capacitor_THT:C_Rect_L7.2mm_W5.5mm_P5.00mm_FKS2_FKP2_MKS2_MKP2
- C12, C13: value 47pF -> 47pF PP; footprint Capacitor_THT:C_Disc_D5.0mm_W2.5mm_P5.00mm -> Capacitor_THT:C_Rect_L7.2mm_W4.5mm_P5.00mm_FKS2_FKP2_MKS2_MKP2
- C15: footprint Capacitor_THT:C_Rect_L7.0mm_W3.5mm_P5.00mm -> Capacitor_THT:C_Rect_L7.2mm_W5.5mm_P5.00mm_FKS2_FKP2_MKS2_MKP2
- C16, C17: value 10uF -> 10uF 25V
- C2: value 220uF -> 220uF 25V A; footprint Capacitor_THT:CP_Radial_D6.3mm_P2.50mm -> Capacitor_THT:CP_Radial_D8.0mm_P3.50mm
- C3, C6: value 100uF -> 100uF 25V A
- C4, C7: value 100nF -> 100nF PP; footprint Capacitor_THT:C_Rect_L7.0mm_W3.5mm_P5.00mm -> Capacitor_THT:C_Rect_L7.2mm_W4.5mm_P5.00mm_FKS2_FKP2_MKS2_MKP2
- C5, C8: value 6.8nF -> 6.8nF PP
Other:
- moved on the sheet: C18, C19, C20, J1, U1C, U2C
